File: hardware/DotControl.sch (EAGLE design)
At the start: 26 parts, among them CN1 1X4-BIG, J3 USB-MICROB, SW2 Previous, SW5 Previous, SW6 Next, SW8 Ok, U1 ATMEGA328P-MU-QFN32, U2 TMP102, U3 ATSHA204-TSU

Commit message: Add HW support for USB bootloading
Parts:
- added D1, D2: (no value), diode:DIODE-SOD523
- added R3, R4, R5: (no value), rcl:R-EU_R0603
Connections:
- removed net MOVE_INT: SW8.2, U1.PC2(ADC2PCINT10)
- removed net OUTB: SW6.2, U1.PC1(ADC1PCINT9)
- new net D+: R3.2, U1.PC2(ADC2PCINT10)
- new net D-: R4.2, R5.1, U1.PC1(ADC1PCINT9)
- new net USB_D+: D2.C, J3.D+, R3.1
- new net USB_D-: D1.C, J3.D-, R4.1
- net +5V: now also R5.2
- net GND: now also D1.A, D2.A
Changed lines of the file:
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@@
 <part name="SJ2" library="SparkFun" deviceset="SOLDERJUMPER" device="TRACE"/>
 <part name="+3V9" library="supply1" deviceset="+3V3" device=""/>
+<part name="D1" library="diode" deviceset="DIODE-" device="SOD523"/>
+<part name="D2" library="diode" deviceset="DIODE-" device="SOD523"/>
+<part name="SUPPLY14" library="supply2" deviceset="GND" device=""/>
+<part name="R3" library="rcl" deviceset="R-EU_" device="R0603"/>
+<part name="R4" library="rcl" deviceset="R-EU_" device="R0603"/>
+<part name="R5" library="rcl" deviceset="R-EU_" device="R0603"/>
+<part name="P+1" library="supply1" deviceset="+5V" device=""/>
 </parts>
 <sheets>
@@
 <instance part="SUPPLY19" gate="GND" x="62.23" y="229.87" rot="R180"/>
 <instance part="P+3" gate="1" x="111.76" y="205.74" rot="R90"/>
-<instance part="SUPPLY10" gate="GND" x="114.3" y="193.04"/>
+<instance part="SUPPLY10" gate="GND" x="121.92" y="193.04"/>
 <instance part="J3" gate="G$1" x="124.46" y="203.2"/>
 <instance part="U$4" gate="G$1" x="170.18" y="200.66"/>
@@
 <instance part="SJ2" gate="1" x="217.17" y="34.29" rot="R180"/>
 <instance part="+3V9" gate="G$1" x="134.62" y="149.86"/>
+<instance part="D1" gate="G$1" x="322.58" y="99.06" rot="R90"/>
+<instance part="D2" gate="G$1" x="332.74" y="99.06" rot="R90"/>
+<instance part="SUPPLY14" gate="GND" x="322.58" y="88.9" rot="MR0"/>
+<instance part="R3" gate="G$1" x="347.98" y="111.76"/>
+<instance part="R4" gate="G$1" x="347.98" y="109.22"/>
+<instance part="R5" gate="G$1" x="358.14" y="121.92" rot="R90"/>
+<instance part="P+1" gate="1" x="358.14" y="129.54"/>
 </instances>
 <busses>
@@
 </segment>
 <segment>
-<wire x1="121.92" y1="195.58" x2="114.3" y2="195.58" width="0.1524" layer="91"/>
 <pinref part="SUPPLY10" gate="GND" pin="GND"/>
 <pinref part="J3" gate="G$1" pin="GND"/>
@@
 <wire x1="223.52" y1="55.88" x2="228.6" y2="55.88" width="0.1524" layer="91"/>
 <pinref part="SUPPLY5" gate="GND" pin="GND"/>
+</segment>
+<segment>
+<pinref part="D1" gate="G$1" pin="A"/>
+<pinref part="D2" gate="G$1" pin="A"/>
+<wire x1="322.58" y1="96.52" x2="332.74" y2="96.52" width="0.1524" layer="91"/>
+<pinref part="SUPPLY14" gate="GND" pin="GND"/>
+<wire x1="322.58" y1="96.52" x2="322.58" y2="91.44" width="0.1524" layer="91"/>
+<junction x="322.58" y="96.52"/>
 </segment>
 </net>
@@
 <pinref part="P+5" gate="1" pin="+5V"/>
 </segment>
+<segment>
+<pinref part="R5" gate="G$1" pin="2"/>
+<pinref part="P+1" gate="1" pin="+5V"/>
+</segment>
 </net>
 <net name="MOSI" class="0">
@@
 </segment>
 </net>
-<net name="MOVE_INT" class="0">
-<segment>
-<pinref part="U1" gate="G$1" pin="PC2(ADC2PCINT10)"/>
-<wire x1="327.66" y1="208.28" x2="330.2" y2="208.28" width="0.1524" layer="91"/>
-<label x="330.2" y="208.28" size="1.27" layer="95" xref="yes"/>
-</segment>
-<segment>
-<pinref part="SW8" gate="G$1" pin="2"/>
-<wire x1="99.06" y1="60.96" x2="99.06" y2="83.82" width="0.1524" layer="91"/>
-<label x="99.06" y="83.82" size="1.27" layer="95" xref="yes"/>
-</segment>
-</net>
 <net name="RXD" class="0">
 <segment>
@@
 <label x="167.64" y="259.08" size="1.27" layer="95" rot="R270" xref="yes"/>
 <pinref part="R2" gate="C" pin="1"/>
-</segment>
-</net>
-<net name="OUTB" class="0">
-<segment>
-<pinref part="U1" gate="G$1" pin="PC1(ADC1PCINT9)"/>
-<wire x1="327.66" y1="210.82" x2="330.2" y2="210.82" width="0.1524" layer="91"/>
-<label x="330.2" y="210.82" size="1.27" layer="95" xref="yes"/>
-</segment>
-<segment>
-<label x="93.98" y="83.82" size="1.27" layer="95" rot="R90" xref="yes"/>
-<pinref part="SW6" gate="G$1" pin="2"/>
-<wire x1="93.98" y1="83.82" x2="93.98" y2="60.96" width="0.1524" layer="91"/>
 </segment>
 </net>
@@
 </segment>
 </net>
+<net name="USB_D-" class="0">
+<segment>
+<pinref part="D1" gate="G$1" pin="C"/>
+<wire x1="322.58" y1="101.6" x2="322.58" y2="109.22" width="0.1524" layer="91"/>
+<wire x1="322.58" y1="109.22" x2="317.5" y2="109.22" width="0.1524" layer="91"/>
+<label x="317.5" y="109.22" size="1.27" layer="95" rot="R180" xref="yes"/>
+<wire x1="322.58" y1="109.22" x2="342.9" y2="109.22" width="0.1524" layer="91"/>
+<junction x="322.58" y="109.22"/>
+<pinref part="R4" gate="G$1" pin="1"/>
+</segment>
+<segment>
+<pinref part="J3" gate="G$1" pin="D-"/>
+<wire x1="121.92" y1="208.28" x2="114.3" y2="208.28" width="0.1524" layer="91"/>
+<label x="114.3" y="208.28" size="1.27" layer="95" rot="R180" xref="yes"/>
+</segment>
+</net>
+<net name="USB_D+" class="0">
+<segment>
+<pinref part="D2" gate="G$1" pin="C"/>
+<wire x1="332.74" y1="101.6" x2="332.74" y2="111.76" width="0.1524" layer="91"/>
+<wire x1="332.74" y1="111.76" x2="317.5" y2="111.76" width="0.1524" layer="91"/>
+<label x="317.5" y="111.76" size="1.27" layer="95" rot="R180" xref="yes"/>
+<wire x1="332.74" y1="111.76" x2="342.9" y2="111.76" width="0.1524" layer="91"/>
+<junction x="332.74" y="111.76"/>
+<pinref part="R3" gate="G$1" pin="1"/>
+</segment>
+<segment>
+<pinref part="J3" gate="G$1" pin="D+"/>
+<wire x1="121.92" y1="210.82" x2="114.3" y2="210.82" width="0.1524" layer="91"/>
+<label x="114.3" y="210.82" size="1.27" layer="95" rot="R180" xref="yes"/>
+</segment>
+</net>
+<net name="D-" class="0">
+<segment>
+<pinref part="R4" gate="G$1" pin="2"/>
+<wire x1="353.06" y1="109.22" x2="358.14" y2="109.22" width="0.1524" layer="91"/>
+<pinref part="R5" gate="G$1" pin="1"/>
+<wire x1="358.14" y1="109.22" x2="368.3" y2="109.22" width="0.1524" layer="91"/>
+<wire x1="358.14" y1="116.84" x2="358.14" y2="109.22" width="0.1524" layer="91"/>
+<junction x="358.14" y="109.22"/>
+<label x="368.3" y="109.22" size="1.27" layer="95" xref="yes"/>
+</segment>
+<segment>
+<pinref part="U1" gate="G$1" pin="PC1(ADC1PCINT9)"/>
+<wire x1="327.66" y1="210.82" x2="330.2" y2="210.82" width="0.1524" layer="91"/>
+<label x="330.2" y="210.82" size="1.27" layer="95" xref="yes"/>
+</segment>
+</net>
+<net name="D+" class="0">
+<segment>
+<pinref part="R3" gate="G$1" pin="2"/>
+<wire x1="353.06" y1="111.76" x2="368.3" y2="111.76" width="0.1524" layer="91"/>
+<label x="368.3" y="111.76" size="1.27" layer="95" xref="yes"/>
+</segment>
+<segment>
+<pinref part="U1" gate="G$1" pin="PC2(ADC2PCINT10)"/>
+<wire x1="327.66" y1="208.28" x2="330.2" y2="208.28" width="0.1524" layer="91"/>
+<label x="330.2" y="208.28" size="1.27" layer="95" xref="yes"/>
+</segment>
+</net>

Commit message: Reassign push buttons
Connections:
- net ADCENA: now also SW6.2; no longer SW2.2
- net BUZZER: now also SW8.2; no longer SW5.2
- net LED: now also SW5.2
- net TXD: now also SW2.2
Changed lines of the file:
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@@
 <pinref part="R2" gate="D" pin="1"/>
+</segment>
+<segment>
+<pinref part="SW5" gate="G$1" pin="2"/>
+<wire x1="88.9" y1="60.96" x2="88.9" y2="71.12" width="0.1524" layer="91"/>
+<label x="88.9" y="71.12" size="1.27" layer="95" rot="R90" xref="yes"/>
 </segment>
 </net>
@@
 </segment>
 <segment>
-<label x="83.82" y="83.82" size="1.27" layer="95" rot="R90" xref="yes"/>
-<pinref part="SW2" gate="G$1" pin="2"/>
-<wire x1="83.82" y1="83.82" x2="83.82" y2="60.96" width="0.1524" layer="91"/>
-</segment>
-<segment>
 <pinref part="U3" gate="G$1" pin="SDA"/>
 <wire x1="205.74" y1="58.42" x2="200.66" y2="58.42" width="0.1524" layer="91"/>
 <label x="200.66" y="58.42" size="1.27" layer="95" rot="R180" xref="yes"/>
+</segment>
+<segment>
+<pinref part="SW6" gate="G$1" pin="2"/>
+<wire x1="93.98" y1="60.96" x2="93.98" y2="71.12" width="0.1524" layer="91"/>
+<label x="93.98" y="71.12" size="1.27" layer="95" rot="R90" xref="yes"/>
 </segment>
 </net>
@@
 <label x="177.8" y="259.08" size="1.27" layer="95" rot="R270" xref="yes"/>
 <pinref part="R2" gate="B" pin="1"/>
+</segment>
+<segment>
+<pinref part="SW2" gate="G$1" pin="2"/>
+<wire x1="83.82" y1="60.96" x2="83.82" y2="71.12" width="0.1524" layer="91"/>
+<label x="83.82" y="71.12" size="1.27" layer="95" rot="R90" xref="yes"/>
 </segment>
 </net>
@@
 </segment>
 <segment>
-<pinref part="SW5" gate="G$1" pin="2"/>
-<wire x1="88.9" y1="60.96" x2="88.9" y2="83.82" width="0.1524" layer="91"/>
-<label x="88.9" y="83.82" size="1.27" layer="95" rot="R90" xref="yes"/>
+<pinref part="SW8" gate="G$1" pin="2"/>
+<wire x1="99.06" y1="60.96" x2="99.06" y2="71.12" width="0.1524" layer="91"/>
+<label x="99.06" y="71.12" size="1.27" layer="95" rot="R90" xref="yes"/>
 </segment>
 </net>

Commit message: Setting vias near rgb R-array further apart
Parts:
- added X1: (no value), adafruit:ANTENNA_U.FL
Connections:
- new net N$3: U$1.ANT, X1.SIGNAL
- net GND: now also X1.GND@0, X1.GND@1
Changed lines of the file:
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@@
 <part name="R5" library="rcl" deviceset="R-EU_" device="R0603"/>
 <part name="P+1" library="supply1" deviceset="+5V" device=""/>
+<part name="X1" library="adafruit" deviceset="ANTENNA_U.FL" device=""/>
+<part name="SUPPLY9" library="supply2" deviceset="GND" device=""/>
 </parts>
 <sheets>
@@
 <instance part="R5" gate="G$1" x="358.14" y="121.92" rot="R90"/>
 <instance part="P+1" gate="1" x="358.14" y="129.54"/>
+<instance part="X1" gate="G$1" x="419.1" y="223.52" rot="R180"/>
+<instance part="SUPPLY9" gate="GND" x="424.18" y="226.06"/>
 </instances>
 <busses>
@@
 <wire x1="322.58" y1="96.52" x2="322.58" y2="91.44" width="0.1524" layer="91"/>
 <junction x="322.58" y="96.52"/>
+</segment>
+<segment>
+<pinref part="X1" gate="G$1" pin="GND@0"/>
+<pinref part="SUPPLY9" gate="GND" pin="GND"/>
+<wire x1="421.64" y1="228.6" x2="424.18" y2="228.6" width="0.1524" layer="91"/>
+<pinref part="X1" gate="G$1" pin="GND@1"/>
+<wire x1="421.64" y1="231.14" x2="424.18" y2="231.14" width="0.1524" layer="91"/>
+<wire x1="424.18" y1="231.14" x2="424.18" y2="228.6" width="0.1524" layer="91"/>
+<junction x="424.18" y="228.6"/>
 </segment>
 </net>
@@
 </segment>
 </net>
+<net name="N$3" class="0">
+<segment>
+<pinref part="X1" gate="G$1" pin="SIGNAL"/>
+<wire x1="408.94" y1="223.52" x2="414.02" y2="223.52" width="0.1524" layer="91"/>
+<pinref part="U$1" gate="G$1" pin="ANT"/>
+</segment>
+</net>
