File: hardware/DotControl.brd (EAGLE design)
At the start: 30.7 x 65 mm, 26 parts, among them CN1 1X4-BIG, J3 USB-MICROB, SW2 Previous, SW5 Previous, SW6 Next, SW8 Ok, U1 ATMEGA328P-MU-QFN32, U2 TMP102, U3 ATSHA204-TSU

Commit message: Add HW support for USB bootloading
Parts:
- added D1, D2: (no value), diode:SOD523
- added R3, R4, R5: (no value), rcl:R0603
Connections:
- removed net MOVE_INT: SW8.2, U1.25
- removed net OUTB: SW6.2, U1.24
- new net D+: R3.2, U1.25
- new net D-: R4.2, R5.1, U1.24
- new net USB_D+: D2.C, J3.D+, R3.1
- new net USB_D-: D1.C, J3.D-, R4.1
- net +5V: now also R5.2
- net GND: now also D1.A, D2.A
Routing:
- net MOVE_INT: track 67.6 -> 0.00 mm, vias 1 -> 0
- net D-: track 0.00 -> 43.3 mm, vias 0 -> 8
- net OUTB: track 36.7 -> 0.00 mm, vias 3 -> 0
- net USB_D+: track 0.00 -> 27.5 mm, vias 0 -> 2
- net D+: track 0.00 -> 26.8 mm, vias 0 -> 4
- net USB_D-: track 0.00 -> 21.8 mm
- net GND: track 31.5 -> 38.9 mm, vias 103 -> 104
- net +3V3: track 187.1 -> 189.8 mm
- net RSDI: track 54.4 -> 52.0 mm
- net RIRQ: track 20.6 -> 22.2 mm
- net BUZZER: track 47.6 -> 48.5 mm
- net RSDO: track 37.7 -> 38.6 mm
- net LED: track 60.9 -> 61.5 mm
Other:
- outline, holes or cut-outs redrawn
- board text added: "TODO:!!Multiplex pushbuttons.. See http://www.instructables.com/id/How-to-access-5-buttons-through-1-Arduino-input/"
- board text removed: "Add USB bootloader connections. See http://www.instructables.com/id/How-to-access-5-buttons-through-1-Arduino-input/"

Commit message: Reassign push buttons
Connections:
- net ADCENA: now also SW6.2; no longer SW2.2
- net BUZZER: now also SW8.2; no longer SW5.2
- net LED: now also SW5.2
- net TXD: now also SW2.2
Routing:
- net TXD: track 45.1 -> 61.8 mm, vias 2 -> 4
- net LED: track 61.5 -> 69.2 mm
- net ADCENA: track 81.5 -> 77.4 mm, vias 6 -> 8
- net BUZZER: track 48.5 -> 50.4 mm
Other:
- board text removed: "Display should be 3.3V compatible. Check if solderjumper J1 on it should be soldered to bypass voltage regulator."
- board text removed: "TODO:!!Multiplex pushbuttons.. See http://www.instructables.com/id/How-to-access-5-buttons-through-1-Arduino-input/"
Changed lines of the file:
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@@
 <text x="3.2258" y="36.576" size="1.4224" layer="22" font="vector" rot="MR90" align="center">Mihai Galos
 12.2017</text>
-<text x="-10.4648" y="71.0438" size="1.778" layer="21">Display should be 3.3V compatible. Check if solderjumper J1
-on it should be soldered to bypass voltage regulator.</text>
 <wire x1="1.1684" y1="0" x2="0" y2="1.1176" width="0.001" layer="20" curve="-90"/>
 <wire x1="30.7086" y1="1.1684" x2="29.591" y2="0" width="0.001" layer="20" curve="-90"/>
@@
 <rectangle x1="0.1524" y1="25.527" x2="5.6388" y2="48.9204" layer="41"/>
 <rectangle x1="0.1524" y1="25.527" x2="5.6134" y2="48.9712" layer="42"/>
-<text x="-3.3782" y="84.201" size="1.778" layer="21">TODO:!!Multiplex pushbuttons.. See http://www.instructables.com/id/How-to-access-5-buttons-through-1-Arduino-input/</text>
-<text x="1.7526" y="94.6404" size="1.778" layer="21">Check USB charging</text>
+<text x="4.1402" y="76.581" size="1.778" layer="21">Check USB charging</text>
 </plain>
 <attributes>
@@
 <wire x1="15.6972" y1="55.0164" x2="14.7828" y2="54.102" width="0.1524" layer="1"/>
 <wire x1="19.9644" y1="55.0164" x2="15.6972" y2="55.0164" width="0.1524" layer="1"/>
-<wire x1="21.9456" y1="53.0352" x2="19.9644" y2="55.0164" width="0.1524" layer="1"/>
+<wire x1="21.9456" y1="53.0352" x2="20.9169" y2="54.0639" width="0.1524" layer="1"/>
+<wire x1="20.9169" y1="54.0639" x2="19.9644" y2="55.0164" width="0.1524" layer="1"/>
 <wire x1="21.9456" y1="52.578" x2="21.9456" y2="53.0352" width="0.1524" layer="1"/>
 <wire x1="22.5552" y1="51.9684" x2="21.9456" y2="52.578" width="0.1524" layer="1"/>
@@
 <wire x1="25.3238" y1="30.7848" x2="27.1526" y2="32.6136" width="0.1524" layer="1"/>
 <wire x1="27.1526" y1="32.6136" x2="27.1526" y2="42.1894" width="0.1524" layer="1"/>
+<contactref element="SW5" pad="2"/>
+<wire x1="23" y1="60.625" x2="21.1836" y2="58.8086" width="0.1524" layer="1"/>
+<wire x1="21.1836" y1="58.8086" x2="21.1836" y2="55.5752" width="0.1524" layer="1"/>
+<wire x1="21.1836" y1="55.5752" x2="21.4884" y2="55.2704" width="0.1524" layer="1"/>
+<wire x1="21.4884" y1="55.2704" x2="21.4884" y2="54.6354" width="0.1524" layer="1"/>
+<wire x1="21.4884" y1="54.6354" x2="20.9169" y2="54.0639" width="0.1524" layer="1"/>
 </signal>
 <signal name="LIGHT_SENSE">
@@
 <signal name="ADCENA">
 <contactref element="U1" pad="13"/>
-<contactref element="SW2" pad="2"/>
 <wire x1="11.1252" y1="11.43" x2="13.2842" y2="11.43" width="0.1524" layer="16"/>
 <wire x1="13.2842" y1="11.43" x2="14.4018" y2="11.43" width="0.1524" layer="16"/>
 <wire x1="10.668" y1="11.8872" x2="11.1252" y2="11.43" width="0.1524" layer="16"/>
 <wire x1="10.3632" y1="26.2128" x2="9.144" y2="24.9936" width="0.1524" layer="16"/>
-<wire x1="10.3632" y1="46.7868" x2="10.3632" y2="26.2128" width="0.1524" layer="1"/>
-<wire x1="4.8768" y1="52.2732" x2="10.3632" y2="46.7868" width="0.1524" layer="1"/>
-<wire x1="4.7244" y1="52.2732" x2="4.8768" y2="52.2732" width="0.1524" layer="1"/>
-<wire x1="4.2672" y1="52.7304" x2="4.7244" y2="52.2732" width="0.1524" layer="1"/>
-<wire x1="3.9624" y1="52.7304" x2="4.2672" y2="52.7304" width="0.1524" layer="1"/>
-<wire x1="3.5052" y1="53.1876" x2="3.9624" y2="52.7304" width="0.1524" layer="1"/>
-<wire x1="3.5052" y1="54.2544" x2="3.5052" y2="53.1876" width="0.1524" layer="1"/>
-<wire x1="4.572" y1="55.3212" x2="3.5052" y2="54.2544" width="0.1524" layer="1"/>
-<wire x1="6.2484" y1="55.3212" x2="4.572" y2="55.3212" width="0.1524" layer="1"/>
-<wire x1="7.62" y1="53.9496" x2="6.2484" y2="55.3212" width="0.1524" layer="1"/>
+<wire x1="10.3632" y1="47.8282" x2="10.3632" y2="26.2128" width="0.1524" layer="1"/>
 <wire x1="14.859" y1="15.5702" x2="14.85" y2="15.6" width="0.1524" layer="16"/>
-<wire x1="7.62" y1="53.9496" x2="7.7" y2="54.075" width="0.1524" layer="1"/>
 <via x="10.668" y="11.8872" extent="1-16" drill="0.3"/>
 <via x="9.144" y="24.9936" extent="1-16" drill="0.3"/>
@@
 <wire x1="10.6172" y1="16.3576" x2="10.6172" y2="11.938" width="0.1524" layer="1"/>
 <wire x1="10.6172" y1="11.938" x2="10.668" y2="11.8872" width="0.1524" layer="1"/>
+<contactref element="SW6" pad="2"/>
+<wire x1="18.925" y1="51.9" x2="17.3404" y2="51.9" width="0.1524" layer="1"/>
+<wire x1="17.3404" y1="51.9" x2="16.764" y2="52.4764" width="0.1524" layer="1"/>
+<via x="16.764" y="52.4764" extent="1-16" drill="0.3" shape="octagon"/>
+<wire x1="16.764" y1="52.4764" x2="15.0114" y2="52.4764" width="0.1524" layer="16"/>
+<wire x1="15.0114" y1="52.4764" x2="10.7696" y2="48.2346" width="0.1524" layer="16"/>
+<via x="10.7696" y="48.2346" extent="1-16" drill="0.3"/>
+<wire x1="10.7696" y1="48.2346" x2="10.3632" y2="47.8282" width="0.1524" layer="1"/>
 </signal>
 <signal name="TXD">
@@
 <wire x1="19.9644" y1="54.102" x2="16.6116" y2="54.102" width="0.1524" layer="1"/>
 <wire x1="21.336" y1="52.7304" x2="19.9644" y2="54.102" width="0.1524" layer="1"/>
-<wire x1="21.336" y1="47.0916" x2="21.336" y2="52.7304" width="0.1524" layer="1"/>
+<wire x1="21.336" y1="47.0916" x2="21.336" y2="48.5648" width="0.1524" layer="1"/>
+<wire x1="21.336" y1="48.5648" x2="21.336" y2="52.7304" width="0.1524" layer="1"/>
 <wire x1="26.5176" y1="41.91" x2="21.336" y2="47.0916" width="0.1524" layer="1"/>
 <wire x1="26.5176" y1="33.3756" x2="26.5176" y2="41.91" width="0.1524" layer="1"/>
@@
 <via x="16.6116" y="54.102" extent="1-16" drill="0.3"/>
 <via x="16.6116" y="21.6408" extent="1-16" drill="0.3"/>
+<contactref element="SW2" pad="2"/>
+<wire x1="7.7" y1="54.075" x2="9.5266" y2="54.075" width="0.1524" layer="1"/>
+<wire x1="9.5266" y1="54.075" x2="10.3124" y2="53.2892" width="0.1524" layer="1"/>
+<wire x1="10.3124" y1="53.2892" x2="13.716" y2="53.2892" width="0.1524" layer="1"/>
+<via x="20.5486" y="48.514" extent="1-16" drill="0.3"/>
+<wire x1="20.5486" y1="48.514" x2="21.2852" y2="48.514" width="0.1524" layer="1"/>
+<wire x1="21.2852" y1="48.514" x2="21.336" y2="48.5648" width="0.1524" layer="1"/>
+<wire x1="18.1356" y1="48.514" x2="18.0848" y2="48.4632" width="0.1524" layer="1"/>
+<wire x1="13.716" y1="53.2892" x2="18.0848" y2="48.9204" width="0.1524" layer="1"/>
+<wire x1="18.0848" y1="48.9204" x2="18.0848" y2="48.4632" width="0.1524" layer="1"/>
+<wire x1="20.5486" y1="48.514" x2="18.8214" y2="48.514" width="0.1524" layer="16"/>
+<wire x1="18.8214" y1="48.514" x2="18.0848" y2="48.4886" width="0.1524" layer="16"/>
+<via x="18.0848" y="48.4886" extent="1-16" drill="0.3"/>
+<wire x1="18.0848" y1="48.4886" x2="18.2118" y2="48.3362" width="0.1524" layer="1"/>
+<wire x1="18.2118" y1="48.3362" x2="18.0848" y2="48.4632" width="0.1524" layer="1"/>
 </signal>
 <signal name="RXD">
@@
 <signal name="BUZZER">
 <contactref element="U1" pad="23"/>
-<contactref element="SW5" pad="2"/>
 <wire x1="11.43" y1="19.3548" x2="12.4968" y2="19.3548" width="0.1524" layer="16"/>
 <wire x1="10.9728" y1="19.812" x2="11.43" y2="19.3548" width="0.1524" layer="16"/>
@@
 <wire x1="11.43" y1="24.9936" x2="10.9728" y2="24.5364" width="0.1524" layer="16"/>
 <wire x1="20.8788" y1="55.0164" x2="15.5448" y2="49.6824" width="0.1524" layer="16"/>
-<wire x1="20.8788" y1="56.9976" x2="20.8788" y2="55.0164" width="0.1524" layer="1"/>
-<wire x1="22.7076" y1="58.8264" x2="20.8788" y2="56.9976" width="0.1524" layer="1"/>
-<wire x1="22.7076" y1="60.3504" x2="22.7076" y2="58.8264" width="0.1524" layer="1"/>
-<wire x1="22.86" y1="60.5028" x2="22.7076" y2="60.3504" width="0.1524" layer="1"/>
 <wire x1="12.4968" y1="19.3548" x2="12.6" y2="19.35" width="0.1524" layer="16"/>
-<wire x1="22.86" y1="60.5028" x2="23" y2="60.625" width="0.1524" layer="1"/>
 <via x="11.43" y="24.9936" extent="1-16" drill="0.3"/>
 <via x="15.5448" y="49.6824" extent="1-16" drill="0.3"/>
@@
 <wire x1="11.4808" y1="26.5684" x2="11.4808" y2="25.0444" width="0.1524" layer="1"/>
 <wire x1="11.4808" y1="25.0444" x2="11.43" y2="24.9936" width="0.1524" layer="1"/>
+<contactref element="SW8" pad="2"/>
+<wire x1="20.8788" y1="55.0164" x2="20.8788" y2="60.759" width="0.1524" layer="1"/>
+<wire x1="20.8788" y1="60.759" x2="19.0266" y2="62.6112" width="0.1524" layer="1"/>
 </signal>
 <signal name="OUTA">

Commit message: Setting vias near rgb R-array further apart
Parts:
- added X1: (no value), adafruit:U.FL
Connections:
- new net N$3: U$1.ANT, X1.3
- net GND: now also X1.1, X1.2
Routing:
- net N$3: track 0.00 -> 2.79 mm, vias 0 -> 1
- net N$10: track 18.3 -> 19.1 mm
- net TXD: track 61.8 -> 62.4 mm
Changed lines of the file:
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@@
 <layer number="20" name="Dimension" color="15" fill="1" visible="yes" active="yes"/>
 <layer number="21" name="tPlace" color="7" fill="1" visible="yes" active="yes"/>
-<layer number="22" name="bPlace" color="7" fill="1" visible="no" active="yes"/>
+<layer number="22" name="bPlace" color="7" fill="1" visible="yes" active="yes"/>
 <layer number="23" name="tOrigins" color="15" fill="1" visible="yes" active="yes"/>
 <layer number="24" name="bOrigins" color="15" fill="1" visible="yes" active="yes"/>
@@
 <layer number="39" name="tKeepout" color="4" fill="11" visible="no" active="yes"/>
 <layer number="40" name="bKeepout" color="1" fill="11" visible="no" active="yes"/>
-<layer number="41" name="tRestrict" color="4" fill="10" visible="yes" active="yes"/>
-<layer number="42" name="bRestrict" color="1" fill="10" visible="yes" active="yes"/>
+<layer number="41" name="tRestrict" color="4" fill="10" visible="no" active="yes"/>
+<layer number="42" name="bRestrict" color="1" fill="10" visible="no" active="yes"/>
 <layer number="43" name="vRestrict" color="2" fill="10" visible="no" active="yes"/>
 <layer number="44" name="Drills" color="7" fill="1" visible="no" active="yes"/>
@@
 <layer number="46" name="Milling" color="3" fill="1" visible="no" active="yes"/>
 <layer number="47" name="Measures" color="7" fill="1" visible="no" active="yes"/>
-<layer number="48" name="Document" color="7" fill="1" visible="yes" active="yes"/>
+<layer number="48" name="Document" color="7" fill="1" visible="no" active="yes"/>
 <layer number="49" name="Reference" color="7" fill="1" visible="no" active="yes"/>
 <layer number="50" name="dxf" color="7" fill="1" visible="no" active="no"/>
@@
 <element name="R4" library="rcl" package="R0603" value="" x="27.8638" y="25.8318" rot="MR90"/>
 <element name="R5" library="rcl" package="R0603" value="" x="27.8638" y="32.6644" rot="MR90"/>
+<element name="X1" library="adafruit" package="U.FL" value="" x="3.9624" y="26.7208"/>
 </elements>
 <signals>
@@
 <via x="4" y="49.5" extent="1-16" drill="0.3"/>
 <via x="6.3" y="49.5" extent="1-16" drill="0.3"/>
-<via x="0.9" y="24.6" extent="1-16" drill="0.3"/>
+<via x="0.9254" y="25.0572" extent="1-16" drill="0.3"/>
 <via x="0.9" y="22.2" extent="1-16" drill="0.3"/>
 <via x="0.9" y="19.9" extent="1-16" drill="0.3"/>
@@
 <wire x1="19.7476" y1="11.1252" x2="19.7476" y2="9.9276" width="0.1524" layer="16"/>
 <wire x1="19.7476" y1="9.9276" x2="18.82" y2="9" width="0.1524" layer="16"/>
-<via x="3.9988" y="24.6762" extent="1-16" drill="0.3"/>
+<via x="3.9988" y="25.1588" extent="1-16" drill="0.3"/>
 <wire x1="17.6" y1="17.85" x2="16.7578" y2="17.85" width="0.1524" layer="16"/>
 <wire x1="16.7578" y1="17.85" x2="15.9258" y2="17.018" width="0.1524" layer="16"/>
@@
 <via x="24.3586" y="25.8572" extent="1-16" drill="0.3"/>
 <wire x1="24.2014" y1="25.7" x2="24.3586" y2="25.8572" width="0.1524" layer="1"/>
-<via x="7.0214" y="24.6254" extent="1-16" drill="0.3"/>
+<via x="6.996" y="25.1334" extent="1-16" drill="0.3"/>
 <via x="13.8032" y="27.4956" extent="1-16" drill="0.3"/>
 <via x="12.2792" y="35.4712" extent="1-16" drill="0.3"/>
@@
 <via x="25.6904" y="34.8616" extent="1-16" drill="0.3"/>
 <via x="24.5686" y="41.2904" extent="1-16" drill="0.3"/>
+<contactref element="X1" pad="1"/>
+<contactref element="X1" pad="2"/>
 <wire x1="16.256" y1="17.85" x2="16.1798" y2="17.8308" width="0" layer="19" extent="16-16"/>
+<wire x1="3.9624" y1="28.0958" x2="3.9624" y2="25.3458" width="0" layer="19" extent="1-1"/>
 </signal>
 <signal name="SCK">
@@
 <wire x1="14.478" y1="54.102" x2="14.478" y2="54.4068" width="0.1524" layer="16"/>
 <wire x1="14.7828" y1="54.102" x2="14.478" y2="54.102" width="0.1524" layer="1"/>
-<wire x1="15.6972" y1="55.0164" x2="14.7828" y2="54.102" width="0.1524" layer="1"/>
-<wire x1="19.9644" y1="55.0164" x2="15.6972" y2="55.0164" width="0.1524" layer="1"/>
+<wire x1="15.6464" y1="55.0672" x2="14.7828" y2="54.102" width="0.1524" layer="1"/>
+<wire x1="19.9136" y1="55.0672" x2="15.6464" y2="55.0672" width="0.1524" layer="1"/>
 <wire x1="21.9456" y1="53.0352" x2="20.9169" y2="54.0639" width="0.1524" layer="1"/>
-<wire x1="20.9169" y1="54.0639" x2="19.9644" y2="55.0164" width="0.1524" layer="1"/>
+<wire x1="20.9169" y1="54.0639" x2="19.9136" y2="55.0672" width="0.1524" layer="1"/>
 <wire x1="21.9456" y1="52.578" x2="21.9456" y2="53.0352" width="0.1524" layer="1"/>
 <wire x1="22.5552" y1="51.9684" x2="21.9456" y2="52.578" width="0.1524" layer="1"/>
@@
 <contactref element="R2" pad="2"/>
 <wire x1="16.1544" y1="54.5592" x2="16.1544" y2="54.864" width="0.1524" layer="16"/>
-<wire x1="16.6116" y1="54.102" x2="16.1544" y2="54.5592" width="0.1524" layer="16"/>
-<wire x1="19.9644" y1="54.102" x2="16.6116" y2="54.102" width="0.1524" layer="1"/>
-<wire x1="21.336" y1="52.7304" x2="19.9644" y2="54.102" width="0.1524" layer="1"/>
+<wire x1="16.764" y1="53.7464" x2="16.1544" y2="54.5592" width="0.1524" layer="16"/>
+<wire x1="19.685" y1="54.356" x2="17.653" y2="54.356" width="0.1524" layer="1"/>
+<wire x1="17.653" y1="54.356" x2="17.0942" y2="53.7464" width="0.1524" layer="1"/>
+<wire x1="17.0942" y1="53.7464" x2="16.764" y2="53.7464" width="0.1524" layer="1"/>
+<wire x1="21.336" y1="52.7304" x2="19.685" y2="54.356" width="0.1524" layer="1"/>
 <wire x1="21.336" y1="47.0916" x2="21.336" y2="48.5648" width="0.1524" layer="1"/>
 <wire x1="21.336" y1="48.5648" x2="21.336" y2="52.7304" width="0.1524" layer="1"/>
@@
 <wire x1="16.1544" y1="54.864" x2="16.2" y2="54.975" width="0.1524" layer="16"/>
 <wire x1="16.3068" y1="20.7264" x2="16.35" y2="20.6" width="0.1524" layer="16"/>
-<via x="16.6116" y="54.102" extent="1-16" drill="0.3"/>
+<via x="16.764" y="53.7464" extent="1-16" drill="0.3"/>
 <via x="16.6116" y="21.6408" extent="1-16" drill="0.3"/>
 <contactref element="SW2" pad="2"/>
@@
 <contactref element="U1" pad="30"/>
 <contactref element="R2" pad="3"/>
-<wire x1="15.3924" y1="54.4068" x2="15.3924" y2="54.864" width="0.1524" layer="16"/>
-<wire x1="15.6972" y1="54.102" x2="15.3924" y2="54.4068" width="0.1524" layer="16"/>
-<wire x1="16.3068" y1="54.7116" x2="15.6972" y2="54.102" width="0.1524" layer="1"/>
-<wire x1="19.812" y1="54.7116" x2="16.3068" y2="54.7116" width="0.1524" layer="1"/>
+<wire x1="15.4178" y1="54.0512" x2="15.3924" y2="54.864" width="0.1524" layer="16"/>
+<wire x1="15.5956" y1="53.7718" x2="15.4178" y2="54.0512" width="0.1524" layer="16"/>
+<wire x1="16.5354" y1="54.7116" x2="15.5956" y2="53.7718" width="0.1524" layer="1"/>
+<wire x1="19.812" y1="54.7116" x2="16.5354" y2="54.7116" width="0.1524" layer="1"/>
 <wire x1="21.6408" y1="52.8828" x2="19.812" y2="54.7116" width="0.1524" layer="1"/>
 <wire x1="21.6408" y1="47.244" x2="21.6408" y2="52.8828" width="0.1524" layer="1"/>
@@
 <wire x1="15.3924" y1="54.864" x2="15.4" y2="54.975" width="0.1524" layer="16"/>
 <wire x1="15.8496" y1="20.7264" x2="15.85" y2="20.6" width="0.1524" layer="16"/>
-<via x="15.6972" y="54.102" extent="1-16" drill="0.3"/>
+<via x="15.5956" y="53.7718" extent="1-16" drill="0.3"/>
 <via x="17.526" y="23.4696" extent="1-16" drill="0.3"/>
 </signal>
@@
 <contactref element="LED1" pad="1"/>
 <contactref element="R2" pad="5"/>
-<wire x1="13.716" y1="56.2356" x2="14.478" y2="56.2356" width="0.1524" layer="16"/>
-<wire x1="13.716" y1="57.15" x2="13.716" y2="56.2356" width="0.1524" layer="1"/>
-<wire x1="9.4488" y1="61.4172" x2="13.716" y2="57.15" width="0.1524" layer="1"/>
+<wire x1="12.9032" y1="56.2356" x2="14.478" y2="56.2356" width="0.1524" layer="16"/>
+<wire x1="12.9032" y1="57.531" x2="12.9032" y2="56.2356" width="0.1524" layer="1"/>
+<wire x1="9.4488" y1="61.4172" x2="12.9032" y2="57.531" width="0.1524" layer="1"/>
 <wire x1="9.4488" y1="62.3316" x2="9.4488" y2="61.4172" width="0.1524" layer="1"/>
 <wire x1="8.6868" y1="63.0936" x2="9.4488" y2="62.3316" width="0.1524" layer="1"/>
@@
 <wire x1="14.478" y1="56.2356" x2="14.6" y2="56.225" width="0.1524" layer="16"/>
 <wire x1="4.1148" y1="62.0268" x2="4.0775" y2="61.9" width="0.1524" layer="1"/>
-<via x="13.716" y="56.2356" extent="1-16" drill="0.3"/>
+<via x="12.9032" y="56.2356" extent="1-16" drill="0.3"/>
 </signal>
 <signal name="N$10">
@@
 <wire x1="15.5448" y1="56.9976" x2="15.5448" y2="56.2356" width="0.1524" layer="16"/>
 <wire x1="15.0876" y1="57.4548" x2="15.5448" y2="56.9976" width="0.1524" layer="16"/>
-<wire x1="14.0208" y1="57.4548" x2="15.0876" y2="57.4548" width="0.1524" layer="16"/>
-<wire x1="10.668" y1="54.102" x2="14.0208" y2="57.4548" width="0.1524" layer="16"/>
 <wire x1="10.0584" y1="54.102" x2="10.668" y2="54.102" width="0.1524" layer="1"/>
 <wire x1="5.4864" y1="58.674" x2="10.0584" y2="54.102" width="0.1524" layer="1"/>
@@
 <wire x1="3.048" y1="60.0456" x2="3.125" y2="60.1" width="0.1524" layer="1"/>
 <via x="10.668" y="54.102" extent="1-16" drill="0.3"/>
+<wire x1="15.0876" y1="57.4548" x2="12.6238" y2="57.4548" width="0.1524" layer="16"/>
+<wire x1="12.6238" y1="57.4548" x2="10.668" y2="55.499" width="0.1524" layer="16"/>
+<wire x1="10.668" y1="55.499" x2="10.668" y2="54.102" width="0.1524" layer="16"/>
 </signal>
 <signal name="N$2">
@@
 <wire x1="21.9964" y1="32.0802" x2="19.3802" y2="32.0802" width="0.1524" layer="16"/>
 </signal>
+<signal name="N$3">
+<contactref element="X1" pad="3"/>
+<contactref element="U$1" pad="ANT"/>
+<wire x1="7.6404" y1="26.7" x2="6.1214" y2="26.7" width="0.4064" layer="16"/>
+<wire x1="6.1214" y1="26.7" x2="6.4262" y2="26.6954" width="0.4064" layer="16"/>
+<via x="6.4262" y="26.6954" extent="1-16" drill="0.3"/>
+<wire x1="6.4262" y1="26.6954" x2="5.4874" y2="26.6954" width="0.4064" layer="1"/>
+<wire x1="5.4874" y1="26.6954" x2="5.4874" y2="26.7208" width="0.4064" layer="1"/>
+</signal>
 </signals>
